File: qwiic-scale.kicad_pcb (KiCad board)
At the start: 4 copper layers, 74.5 x 34.5 mm, 92 parts, among them J1 USB_B_Micro, J10 Conn_01x04, J2 Conn_02x05_Odd_Even, J3 SM04B-SRSS-TB(LF)(SN), J4 SM04B-SRSS-TB(LF)(SN), J5 Conn_01x04, J6 Conn_01x04, J7 Conn_01x04, J8 Conn_01x04, J9 Conn_01x02, SW1 SW_Push, SW2 SW_Push, U1 RP2040, U12 W25Q128JVS, U2 74HCT4066PW, U3 AP3012, U4 AMS1117-3.3, U5 ADS124S08IPBSR, U6 ADP7118, Y1 XYDBPCNANF-12MHZ

Commit message: R1A updates
Parts:
- added D2: D_Schottky, Diode_SMD:D_SOD-323, F.Cu at (64.3, 103.7)
- J2: moved to F.Cu
- moved R6 20.2 mm to (55.0, 101.8), turned to 180 degrees
- moved J1 20.1 mm to (56.8, 104.9)
- moved R5 18.9 mm to (58.2, 101.8), turned to 0 degrees
- moved J9 14.7 mm to (64.1, 115.8), turned to 90 degrees
- moved J2 9.89 mm to (76.3, 113.7), turned to 0 degrees
- moved C33 3.70 mm to (61.6, 101.2)
- moved C34 3.70 mm to (63.9, 101.2)
- moved R4 3.09 mm to (68.0, 105.8), turned to -90 degrees
- moved U6 2.43 mm to (63.4, 98.0)
- moved J5 2.00 mm to (77.0, 86.9)
- moved J6 2.00 mm to (90.1, 86.9)
- moved J7 2.00 mm to (103.1, 86.9)
- moved J8 2.00 mm to (116.0, 86.9)
- moved C9 1.70 mm to (83.6, 111.0), turned to -90 degrees
- moved L1 1.67 mm to (66.0, 111.2)
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Connections:
- C17 pad 2: Net-(U5-REFCOM) -> GND
- C33 pad 2: Net-(U3-SW) -> Net-(D2-K)
- C34 pad 1: Net-(U3-SW) -> Net-(D2-K)
- J5 pad 1: GND -> EXCITATION1
- J5 pad 2: EXCITATION1 -> GND
- J6 pad 1: GND -> EXCITATION2
- J6 pad 2: EXCITATION2 -> GND
- J7 pad 1: GND -> EXCITATION3
- J7 pad 2: EXCITATION3 -> GND
- J8 pad 1: GND -> EXCITATION4
- J8 pad 2: EXCITATION4 -> GND
- L1 pad 2: Net-(U3-SW) -> Net-(D2-A)
- R4 pad 1: Net-(U3-SW) -> Net-(D2-K)
- U3 pad 1: Net-(U3-SW) -> Net-(D2-A)
- U5 pad 15: GND -> QWIIC_VIN
- U5 pad 24: Net-(U5-REFCOM) -> GND
- U6 pad 1: Net-(U3-SW) -> Net-(D2-K)
- U6 pad 3: Net-(U3-SW) -> Net-(D2-K)
Routing:
- net Net-(U3-SW): track 26.9 -> 0.00 mm
- net RP2040_USB_PRE_R_DP: track 18.0 -> 39.6 mm
- net RP2040_USB_PRE_R_DN: track 18.0 -> 39.4 mm
- net GND: track 82.1 -> 98.0 mm, vias 58 -> 55
- net Net-(D2-K): track 0.00 -> 15.7 mm
- net QWIIC_VIN: track 77.8 -> 92.3 mm, vias 18 -> 17
- net RP2040_SWCLK: track 22.4 -> 34.0 mm, vias 1 -> 2
- net RP2040_SWD: track 17.9 -> 29.5 mm, vias 1 -> 2
- net Net-(D2-A): track 0.00 -> 8.97 mm
- net RP2040_RESETn: track 30.5 -> 38.5 mm, vias 1 -> 2
- net RP2040_USB_VBUS: track 31.0 -> 23.1 mm
- net QWIIC_SCL: track 129.0 -> 123.0 mm, vias 2 -> 0
- net EXCITATION1: track 24.3 -> 28.4 mm
- net EXCITATION2: track 16.2 -> 19.3 mm
- net EXCITATION3: track 19.1 -> 21.8 mm
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Other:
- board text added: "Hammond 1551K"
- board text added: "R1A"
- board text removed: "R0A"

Commit message: WIP
Parts:
- moved J4 7.00 mm to (119.9, 113.2)
- moved R10 7.00 mm to (117.6, 111.1)
- moved R9 7.00 mm to (117.6, 113.2)
- moved J8 6.90 mm to (109.1, 86.8)
- moved R8 6.74 mm to (59.5, 91.8)
- moved C36 6.74 mm to (54.0, 101.7)
- moved C39 6.74 mm to (57.6, 101.7)
- moved J1 6.74 mm to (56.3, 98.2)
- moved J3 6.74 mm to (57.2, 89.8)
- moved R5 6.74 mm to (57.8, 95.1)
- moved R6 6.74 mm to (54.6, 95.1)
- moved R7 6.74 mm to (59.5, 89.8)
- moved U4 6.74 mm to (56.7, 106.3)
- moved J7 5.82 mm to (97.3, 86.8)
- moved J6 4.75 mm to (85.4, 86.8)
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Routing:
- net QWIIC_SCL: track 123.0 -> 84.5 mm, vias 0 -> 2
- net QWIIC_SDA: track 125.7 -> 92.3 mm, vias 2 -> 4
- net QWIIC_VIN: track 92.3 -> 66.4 mm, vias 17 -> 25
- net GND: track 98.0 -> 107.9 mm, vias 55 -> 52
- net RP2040_USB_PRE_R_DP: track 39.6 -> 44.4 mm
- net RP2040_USB_PRE_R_DN: track 39.4 -> 44.2 mm
- net RP2040_USB_VBUS: track 23.1 -> 27.1 mm
- net EXCITATION1: track 28.4 -> 31.8 mm
- net Net-(U5-REFOUT): track 1.79 -> 4.59 mm
- net EXCITATION2: track 19.3 -> 21.6 mm
- net EXCITATION3: track 21.8 -> 24.0 mm
- net AVCC: track 96.7 -> 94.7 mm, vias 5 -> 6
- net Net-(J5-Pin_4): track 5.98 -> 7.45 mm
- net Net-(J5-Pin_3): track 5.93 -> 7.40 mm
- net EXCITATION4: track 26.8 -> 28.0 mm
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- added copper zone on In1.Cu, net GND
- added copper zone on F.Cu, net QWIIC_VIN
- added copper zone on In2.Cu, net QWIIC_VIN
- removed copper zone on In2.Cu, net GND
- removed copper zone on In1.Cu, net QWIIC_VIN
Other:
- outline, holes or cut-outs redrawn
- board text added: "R1B"
- board text removed: "R1A"

Commit message: WIP
Parts:
- added C37: 10 µF, Capacitor_SMD:C_0805_2012Metric, F.Cu at (105.7, 100.9)
- added C40: 100 nF, >10V, X6S, Capacitor_SMD:C_0402_1005Metric, F.Cu at (121.9, 98.8)
- added C41: 10 µF, Capacitor_SMD:C_0805_2012Metric, F.Cu at (121.9, 101.2)
- added C42: 100 nF, >10V, X6S, Capacitor_SMD:C_0402_1005Metric, F.Cu at (121.9, 106.6)
- added C43: 10 µF, Capacitor_SMD:C_0805_2012Metric, F.Cu at (122.7, 104.9)
- added C44: 100 nF, >10V, X6S, Capacitor_SMD:C_0402_1005Metric, F.Cu at (92.9, 98.9)
- added J11: Conn_01x02, Connector_PinHeader_2.54mm:PinHeader_1x02_P2.54mm_Vertical, F.Cu at (60.6, 113.1)
- added J12: Conn_01x02, Connector_PinHeader_2.54mm:PinHeader_1x02_P2.54mm_Vertical, F.Cu at (73.6, 90.8)
- added Q7: DMN63D8LDW, PCM_Package_TO_SOT_SMD_AKL:SOT-363_SC-70-6, F.Cu at (97.6, 109.4)
- added Q8: DMN63D8LDW, PCM_Package_TO_SOT_SMD_AKL:SOT-363_SC-70-6, F.Cu at (104.0, 109.3)
- added Q9: DMN63D8LDW, PCM_Package_TO_SOT_SMD_AKL:SOT-363_SC-70-6, F.Cu at (111.3, 110.5)
- added R29: 10K, Resistor_SMD:R_0402_1005Metric, F.Cu at (108.5, 111.2)
- added R30: 10K, Resistor_SMD:R_0402_1005Metric, F.Cu at (106.4, 110.2)
- added R31: 10K, Resistor_SMD:R_0402_1005Metric, F.Cu at (101.7, 110.3)
- C16: value 330 nF -> 10 µF; footprint Capacitor_SMD:C_0603_1608Metric -> Capacitor_SMD:C_0805_2012Metric
- C17: value 1 uF, >10V, X5R -> 100 nF, >10V, X6S
- C19: value 10nF -> 100 nF, >10V, X6S
- C20, C34, C36, C39: value 10µF -> 10 µF
- R20, R21, R22, R23, R24, R25, R26: value 47R -> 10K
- R27, R28: value 100R -> 10K
- U2: value 74HCT4066PW -> NAU7802SGI; footprint Package_SO:SO-14_3.9x8.65mm_P1.27mm -> PCM_Package_SO_AKL:SOP-16_4.4x10.4mm_P1.27mm
- U5: value ADS124S08IPBSR -> NAU7802SGI; footprint Package_QFP:LQFP-32_5x5mm_P0.5mm -> PCM_Package_SO_AKL:SOP-16_4.4x10.4mm_P1.27mm
- moved R26 15.4 mm to (109.0, 109.5), turned to 90 degrees
- moved C18 14.6 mm to (105.7, 98.6), turned to 180 degrees
- moved R25 12.5 mm to (106.4, 108.2), turned to -90 degrees
- moved C17 11.1 mm to (105.9, 106.0), turned to 180 degrees
- moved R28 10.9 mm to (113.7, 111.4)
- moved R27 9.33 mm to (113.7, 109.4), turned to 90 degrees
- moved R24 7.77 mm to (101.7, 108.3), turned to 90 degrees
- moved R21 7.13 mm to (99.9, 108.3), turned to 90 degrees
- moved C16 6.59 mm to (106.7, 104.3)
- moved U5 6.14 mm to (115.2, 103.2), turned to -90 degrees
- moved R22 5.99 mm to (99.9, 110.3), turned to -90 degrees
- moved R20 5.18 mm to (95.3, 108.3), turned to 90 degrees
- moved R3 4.77 mm to (66.7, 95.2), turned to 180 degrees
- moved C19 2.90 mm to (109.0, 99.8), turned to 90 degrees
- moved U2 2.74 mm to (99.0, 102.3), turned to -90 degrees
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Connections:
- net ADS124S08_MOSI renamed NAU7802_1_DRDY_3V3
- C16 pad 1: AVCC -> GND
- C16 pad 2: GND -> AVCC
- C17 pad 1: Net-(U5-REFOUT) -> GND
- C17 pad 2: GND -> AVCC
- C18 pad 1: QWIIC_VIN -> GND
- C18 pad 2: GND -> NAU7802_1_AVDD
- C19 pad 1: REFP0 -> Net-(U5-VBG)
- C19 pad 2: REFN0 -> GND
- J5 pad 1: EXCITATION1 -> NAU7802_1_AVDD
- J6 pad 1: EXCITATION2 -> NAU7802_1_AVDD
- J7 pad 1: EXCITATION3 -> NAU7802_2_AVDD
- J8 pad 1: EXCITATION4 -> NAU7802_2_AVDD
- R20 pad 1: Net-(U5-RESET_N) -> QWIIC_VIN
- R20 pad 2: ADS124S08_RESETn -> NAU7802_1_SDIO_3V3
- R21 pad 1: Net-(U5-DRDY_N) -> AVCC
- R21 pad 2: ADS124S08_DRDY -> NAU7802_1_SDIO_5V
- R22 pad 1: Net-(U5-DOUT_DRDY_N) -> QWIIC_VIN
- R22 pad 2: ADS124S08_MISO -> NAU7802_1_SCLK_3V3
- R23 pad 1: Net-(U5-SCLK) -> AVCC
- R23 pad 2: ADS124S08_SCLK -> NAU7802_1_SCLK_5V
- R24 pad 1: Net-(U5-DIN) -> QWIIC_VIN
- R25 pad 1: Net-(U5-CS_N) -> AVCC
- R25 pad 2: ADS124S08_CS -> NAU7802_1_DRDY_5V
- R26 pad 1: Net-(U5-START_SYNC) -> QWIIC_VIN
- R26 pad 2: ADS124S08_START_SYNC -> NAU7802_2_SDIO_3V3
- R27 pad 2: REFP0 -> NAU7802_2_SDIO_5V
- R28 pad 1: GND -> QWIIC_VIN
- R28 pad 2: REFN0 -> NAU7802_2_SCLK_3V3
- U1 pad 11: ADS124S08_CS -> unconnected-(U1-GPIO8-Pad11)
- U1 pad 12: ADS124S08_START_SYNC -> unconnected-(U1-GPIO9-Pad12)
- U1 pad 13: unconnected-(U1-GPIO10-Pad13) -> NAU7802_1_SDIO_3V3
- U1 pad 14: unconnected-(U1-GPIO11-Pad14) -> NAU7802_1_SCLK_3V3
- U1 pad 15: EXCITATION4_EN -> USER_BUTTON_2
- U1 pad 16: EXCITATION3_EN -> unconnected-(U1-GPIO13-Pad16)
- U1 pad 17: EXCITATION2_EN -> unconnected-(U1-GPIO14-Pad17)
- U1 pad 18: EXCITATION1_EN -> unconnected-(U1-GPIO15-Pad18)
- U1 pad 37: unconnected-(U1-GPIO25-Pad37) -> USER_BUTTON_1
- U1 pad 4: ADS124S08_RESETn -> NAU7802_2_SDIO_3V3
- U1 pad 5: ADS124S08_DRDY -> NAU7802_2_SCLK_3V3
- U1 pad 6: ADS124S08_MISO -> unconnected-(U1-GPIO4-Pad6)
- U1 pad 8: ADS124S08_SCLK -> NAU7802_2_DRDY_3V3
- U2 pad 1: AVCC -> NAU7802_1_AVDD
- U2 pad 10: EXCITATION1 -> unconnected-(U2-XIN-Pad10)
- U2 pad 11: AVCC -> unconnected-(U2-XOUT-Pad11)
- U2 pad 12: EXCITATION1_EN -> NAU7802_1_DRDY_5V
- U2 pad 13: EXCITATION4_EN -> NAU7802_1_SCLK_5V
- U2 pad 14: AVCC -> NAU7802_1_SDIO_5V
- U2 pad 2: EXCITATION4 -> LOAD_CELL_2_N
- U2 pad 3: EXCITATION3 -> LOAD_CELL_2_P
- U2 pad 4: AVCC -> LOAD_CELL_1_N
- U2 pad 5: EXCITATION3_EN -> LOAD_CELL_1_P
- U2 pad 6: EXCITATION2_EN -> Net-(U2-VBG)
- U2 pad 8: AVCC -> GND
- U2 pad 9: EXCITATION2 -> GND
- U5 pad 1: GND -> NAU7802_2_AVDD
- U5 pad 10: Net-(U5-DIN) -> unconnected-(U5-XIN-Pad10)
- U5 pad 11: Net-(U5-SCLK) -> unconnected-(U5-XOUT-Pad11)
- U5 pad 12: Net-(U5-DOUT_DRDY_N) -> NAU7802_2_DRDY_5V
- U5 pad 13: Net-(U5-DRDY_N) -> NAU7802_2_SCLK_5V
- U5 pad 14: GND -> NAU7802_2_SDIO_5V
- U5 pad 15: QWIIC_VIN -> AVCC
- U5 pad 16: QWIIC_VIN -> NAU7802_2_AVDD
- U5 pad 2: LOAD_CELL_2_N -> LOAD_CELL_4_N
- U5 pad 3: LOAD_CELL_2_P -> LOAD_CELL_4_P
- U5 pad 4: unconnected-(U5-AIN3-Pad4) -> LOAD_CELL_3_N
- U5 pad 5: LOAD_CELL_1_N -> LOAD_CELL_3_P
- U5 pad 6: LOAD_CELL_1_P -> Net-(U5-VBG)
- U5 pad 7: unconnected-(U5-AIN0-Pad7) -> GND
- U5 pad 8: Net-(U5-START_SYNC) -> GND
- U5 pad 9: Net-(U5-CS_N) -> GND
Routing:
- net NAU7802_1_AVDD: track 0.00 -> 50.3 mm
- net NAU7802_2_AVDD: track 0.00 -> 44.9 mm, vias 0 -> 1
- net EXCITATION1: track 31.8 -> 0.00 mm, vias 1 -> 0
- net USER_BUTTON_1: track 0.00 -> 31.4 mm
- net USER_BUTTON_2: track 0.00 -> 30.4 mm, vias 0 -> 1
- net EXCITATION4: track 28.0 -> 0.00 mm, vias 1 -> 0
- net Net-(U5-RESET_N): track 25.8 -> 0.00 mm
- net NAU7802_2_SCLK_3V3: track 0.00 -> 24.7 mm, vias 0 -> 2
- net NAU7802_2_SDIO_3V3: track 0.00 -> 24.2 mm, vias 0 -> 2
- net EXCITATION3: track 24.0 -> 0.00 mm, vias 1 -> 0
- net EXCITATION2: track 21.6 -> 0.00 mm, vias 1 -> 0
- net Net-(U5-DRDY_N): track 18.1 -> 0.00 mm
- net LOAD_CELL_1_N: track 40.0 -> 22.6 mm
- net NAU7802_2_DRDY_3V3: track 0.00 -> 17.2 mm
- net Net-(U5-DOUT_DRDY_N): track 17.0 -> 0.00 mm
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Other:
- board text added: "R2A"
- board text removed: "R1B"

Commit message: WIP
Parts:
- removed U6: ADP7118, Package_TO_SOT_SMD:TSOT-23-5
- added C45: 1 nF, Capacitor_SMD:C_0402_1005Metric, F.Cu at (65.9, 97.1)
- added U7: ADM7170ACPZ-1.8-R7, ADM7170ACPZ-1:SON50P300X300X80-9N, F.Cu at (63.2, 98.2)
- C16, C20, C34, C36, C37, C39, C41, C43: value 10 µF -> 10 µF, >10V, X5R
- C21, C22, C24, C25, C27, C28, C30, C31: value 5.1 nF -> X nF
- C23, C26, C29, C32: value 51 nF -> 10X nF
- R11, R12, R13, R14, R15, R16, R17, R18: value 6K04 1% -> Y R
- R19: value 10K -> 6K8; footprint Resistor_SMD:R_0402_1005Metric -> Resistor_SMD:R_0603_1608Metric
- R4: value 47K -> 27K; footprint Resistor_SMD:R_0402_1005Metric -> Resistor_SMD:R_0603_1608Metric
- moved R4 2.45 mm to (66.4, 103.9), turned to 0 degrees
- moved R19 1.41 mm to (68.0, 106.3)
- moved D2 1.16 mm to (63.1, 103.7)
- moved C18 0.73 mm to (106.4, 98.6)
- moved C37 0.73 mm to (106.4, 100.9)
- moved C44 0.72 mm to (92.2, 99.1)
- moved C19 0.67 mm to (108.3, 99.8)
- moved C40 0.66 mm to (122.6, 98.8)
- moved C41 0.66 mm to (122.6, 101.2)
- moved C42 0.66 mm to (122.6, 106.6)
- moved C43 0.66 mm to (123.4, 104.9)
- moved U2 0.57 mm to (99.0, 102.9)
- moved C16 0.36 mm to (107.1, 104.3)
- moved U5 0.33 mm to (115.2, 102.9)
Routing:
- net AVCC: track 107.5 -> 103.2 mm
- net GND: track 112.2 -> 116.4 mm, vias 56 -> 55
- net Net-(D2-K): track 16.1 -> 13.5 mm
- net NAU7802_1_AVDD: track 50.3 -> 51.8 mm
- net Net-(U7-SS): track 0.00 -> 1.32 mm
- net Net-(U3-FB): track 3.01 -> 3.94 mm
- net LOAD_CELL_2_P: track 14.7 -> 15.6 mm
- net LOAD_CELL_1_N: track 22.6 -> 23.5 mm
- net LOAD_CELL_2_N: track 13.3 -> 14.1 mm
- net LOAD_CELL_1_P: track 24.4 -> 25.3 mm
- net NAU7802_1_DRDY_5V: track 11.5 -> 10.6 mm
- net NAU7802_2_AVDD: track 44.9 -> 45.6 mm
- net NAU7802_2_SCLK_5V: track 9.09 -> 9.73 mm
- net NAU7802_2_SDIO_5V: track 6.29 -> 6.94 mm
- net QWIIC_SCL: track 84.6 -> 85.2 mm
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Other:
- board text added: "GP12"
- board text added: "GP25"

Commit message: Final version sent to manufacturing
Parts:
- added D3: KT-0603W, LED_SMD:LED_0603_1608Metric, F.Cu at (85.1, 99.1)
- added JP1: SolderJumper_3_Bridged12, Jumper:SolderJumper-3_P1.3mm_Bridged12_RoundedPad1.0x1.5mm, B.Cu at (98.2, 102.9)
- added R32: 120R, Resistor_SMD:R_0402_1005Metric, F.Cu at (85.6, 100.8)
- added TP1: TestPoint, TestPoint:TestPoint_Pad_D2.0mm, B.Cu at (70.2, 94.9)
- added TP2: TestPoint, TestPoint:TestPoint_Pad_D2.0mm, B.Cu at (70.2, 101.1)
- added TP3: TestPoint, TestPoint:TestPoint_Pad_D1.0mm, B.Cu at (78.0, 111.8)
- added TP4: TestPoint, TestPoint:TestPoint_Pad_D1.0mm, B.Cu at (74.7, 111.8)
- added TP5: TestPoint, TestPoint:TestPoint_Pad_D1.0mm, B.Cu at (78.0, 115.1)
- added TP6: TestPoint, TestPoint:TestPoint_Pad_D1.0mm, B.Cu at (74.7, 115.1)
- C21, C22, C27, C28: value X nF -> DNF
- C23, C29: value 10X nF -> 680 pF, C0G
- C24, C25, C30, C31: value X nF -> 680 pF, C0G
- C26, C32: value 10X nF -> 100 nF, C0G
- C37, C41: value 10 µF, >10V, X5R -> 1 uF, >10V, X5R; footprint Capacitor_SMD:C_0805_2012Metric -> Capacitor_SMD:C_0402_1005Metric
- R11, R12, R15, R16: value Y R -> DNF
- R13, R14, R17, R18: value Y R -> 51R, Precision
- moved REF** 17.6 mm to (118.1, 109.0)
- moved D1 10.2 mm to (88.4, 99.1)
- moved R7 7.97 mm to (66.4, 93.8), turned to 0 degrees
- moved R8 7.78 mm to (66.4, 95.4), turned to 180 degrees
- moved R2 6.35 mm to (87.9, 100.8)
- moved R3 4.27 mm to (69.1, 91.7)
- moved REF** 2.86 mm to (108.5, 103.8)
- moved C7 1.70 mm to (94.0, 112.6)
- moved C41 1.28 mm to (122.6, 99.9), turned to 180 degrees
- moved C37 1.13 mm to (106.4, 99.8), turned to 180 degrees
Connections:
- net LOAD_CELL_1_N renamed LOAD_CELL_ADC1_2_N
- net LOAD_CELL_1_P renamed LOAD_CELL_ADC1_2_P
- net LOAD_CELL_2_N renamed LOAD_CELL_ADC1_1_N
- net LOAD_CELL_2_P renamed LOAD_CELL_ADC1_1_P
- net LOAD_CELL_3_N renamed LOAD_CELL_ADC2_2_N
- net LOAD_CELL_3_P renamed LOAD_CELL_ADC2_2_P
- net LOAD_CELL_4_N renamed LOAD_CELL_ADC2_1_N
- net LOAD_CELL_4_P renamed LOAD_CELL_ADC2_1_P
- C20 pad 1: AVCC -> +5VA
- C35 pad 2: AVCC -> +5VA
- R2 pad 1: Net-(U1-GPIO17) -> Net-(U1-GPIO15)
- U1 pad 17: unconnected-(U1-GPIO14-Pad17) -> Net-(U1-GPIO14)
- U1 pad 18: unconnected-(U1-GPIO15-Pad18) -> Net-(U1-GPIO15)
- U1 pad 27: unconnected-(U1-GPIO16-Pad27) -> Net-(U1-GPIO16)
- U1 pad 29: unconnected-(U1-GPIO18-Pad29) -> Net-(U1-GPIO18)
- U1 pad 30: unconnected-(U1-GPIO19-Pad30) -> Net-(U1-GPIO19)
- U7 pad 1: AVCC -> +5VA
- U7 pad 2: AVCC -> +5VA
- U7 pad 3: AVCC -> +5VA
Routing:
- net +5VA: track 0.00 -> 49.9 mm, vias 0 -> 4
- net AVCC: track 103.2 -> 69.3 mm
- net Net-(U1-GPIO19): track 0.00 -> 20.8 mm, vias 0 -> 1
- net Net-(U1-GPIO16): track 0.00 -> 16.5 mm, vias 0 -> 1
- net Net-(U1-GPIO14): track 0.00 -> 15.9 mm
- net Net-(U1-GPIO17): track 2.70 -> 18.4 mm, vias 0 -> 1
- net Net-(U1-GPIO18): track 0.00 -> 14.4 mm, vias 0 -> 1
- net Net-(D2-K): track 13.5 -> 26.6 mm, vias 0 -> 1
- net Net-(U1-GPIO15): track 0.00 -> 12.2 mm
- net RP2040_USB_PRE_R_DP: track 44.4 -> 55.2 mm
- net RP2040_USB_PRE_R_DN: track 44.2 -> 54.9 mm
- net GND: track 116.4 -> 125.2 mm, vias 55 -> 58
- net NAU7802_1_AVDD: track 51.8 -> 57.8 mm
- net NAU7802_2_AVDD: track 45.6 -> 50.3 mm
- net QWIIC_VIN: track 81.7 -> 86.0 mm, vias 27 -> 32
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Other:
- board text added: "5VA"
- board text added: "6V2"
- board text added: "A1"
- board text added: "A2"
- board text added: "B1"
- board text added: "B2"
- board text added: "GP16"
- board text added: "GP17"
- board text added: "GP18"
- board text added: "GP19"
- board text added: "VUSB"
- board text removed: "5V"

Commit message: WIP
Parts:
- added J13: BM03B-SRSS-TBLFSN, BM03B-SRSS-TB_LF__SN_:CONN_BM03B-SRSS-TBLFSN_JST, F.Cu at (73.1, 113.0)
- added JP2: SolderJumper_3_Bridged12, Jumper:SolderJumper-3_P1.3mm_Bridged12_RoundedPad1.0x1.5mm, B.Cu at (94.2, 111.6)
- added JP3: SolderJumper_3_Bridged12, Jumper:SolderJumper-3_P1.3mm_Bridged12_RoundedPad1.0x1.5mm, B.Cu at (94.2, 108.8)
- added R33: 100R, Resistor_SMD:R_0402_1005Metric, F.Cu at (77.3, 113.9)
- added R34: 100R, Resistor_SMD:R_0402_1005Metric, F.Cu at (77.3, 112.0)
- added TP10: TestPoint_Small, TestPoint:TestPoint_Pad_D1.0mm, B.Cu at (101.6, 106.1)
- added TP11: TestPoint_Small, TestPoint:TestPoint_Pad_D1.0mm, B.Cu at (98.5, 106.1)
- added TP12: TestPoint_Small, TestPoint:TestPoint_Pad_D1.0mm, B.Cu at (95.5, 106.1)
- added TP7: TestPoint_Small, TestPoint:TestPoint_Pad_D1.0mm, B.Cu at (117.8, 110.5)
- added TP8: TestPoint_Small, TestPoint:TestPoint_Pad_D1.0mm, B.Cu at (114.8, 110.5)
- added TP9: TestPoint_Small, TestPoint:TestPoint_Pad_D1.0mm, B.Cu at (111.7, 110.5)
- J2: moved to B.Cu
- moved TP3 13.1 mm to (79.6, 98.8)
- moved TP4 11.6 mm to (79.6, 101.2)
- moved TP5 11.4 mm to (79.6, 103.7)
- moved TP6 10.1 mm to (79.6, 106.2)
- moved J2 1.61 mm to (74.9, 112.9), turned to 180 degrees
Connections:
- U1 pad 11: unconnected-(U1-GPIO8-Pad11) -> NAU7802_1_SDIO_3V3_ALT_B
- U1 pad 12: unconnected-(U1-GPIO9-Pad12) -> NAU7802_1_SCLK_3V3_ALT_B
- U1 pad 13: NAU7802_1_SDIO_3V3 -> NAU7802_1_SDIO_3V3_ALT_A
- U1 pad 14: NAU7802_1_SCLK_3V3 -> NAU7802_1_SCLK_3V3_ALT_A
Routing:
- net Net-(U1-GPIO19): track 20.8 -> 6.44 mm
- net NAU7802_1_DRDY_5V: track 10.6 -> 23.6 mm, vias 0 -> 1
- net NAU7802_1_SDIO_3V3_ALT_A: track 0.00 -> 11.9 mm, vias 0 -> 1
- net NAU7802_1_SCLK_5V: track 6.80 -> 17.0 mm, vias 0 -> 1
- net NAU7802_1_SDIO_3V3_ALT_B: track 0.00 -> 8.90 mm, vias 0 -> 1
- net RP2040_SWCLK: track 34.1 -> 43.0 mm
- net Net-(U1-GPIO17): track 18.4 -> 12.1 mm
- net NAU7802_1_SCLK_3V3_ALT_A: track 0.00 -> 6.06 mm, vias 0 -> 1
- net QWIIC_VIN: track 86.0 -> 91.9 mm, vias 32 -> 31
- net RP2040_SWD: track 29.5 -> 35.2 mm
- net NAU7802_1_SDIO_3V3: track 5.48 -> 11.0 mm, vias 0 -> 1
- net Net-(U1-GPIO18): track 14.4 -> 9.16 mm
- net NAU7802_2_SDIO_5V: track 6.94 -> 11.9 mm, vias 0 -> 1
- net NAU7802_2_SCLK_5V: track 9.18 -> 13.4 mm, vias 0 -> 1
- net NAU7802_1_SDIO_5V: track 3.94 -> 7.93 mm, vias 0 -> 1
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Other:
- board text added: "DBG"
- board text added: "R2B"
- board text added: "Res"
- board text removed: "R2A"
