File: qwiic-scale.kicad_sch (KiCad schematic)
At the start: 90 parts, among them J1 USB_B_Micro, J10 Conn_01x04, J13 Conn_02x05_Odd_Even, J5 Conn_01x04, J5 SM04B-SRSS-TB(LF)(SN), J6 Conn_01x04, J7 Conn_01x04, J8 Conn_01x04, J9 Conn_01x02, SW1 SW_Push, SW2 SW_Push, U12 W25Q128JVS, U2 74HCT4066PW, U2 RP2040, U3 AP3012, U4 AMS1117-3.3, U6 ADP7118, U6 ADS124S08IPBSR, Y1 XYDBPCNANF-12MHZ

Commit message: R1A updates
Parts:
- added D2: D_Schottky, Diode_SMD:D_SOD-323, symbol Device:D_Schottky
- J1, J5: Comment (none) -> Extended
- J10, J5, J6, J7, J8, J9: Comment (none) -> Hand solder
- U4: LCSC (none) -> C6186
Connections:
- net +3V3: now also U6.15 (IOVDD)
- net EXCITATION1: now also J5.1 (Pin_1); no longer J5.2 (Pin_2)
- net EXCITATION2: now also J6.1 (Pin_1); no longer J6.2 (Pin_2)
- net EXCITATION3: now also J7.1 (Pin_1); no longer J7.2 (Pin_2)
- net EXCITATION4: now also J8.1 (Pin_1); no longer J8.2 (Pin_2)
- net GND: now also C47.2, J5.2 (Pin_2), J6.2 (Pin_2), J7.2 (Pin_2), J8.2 (Pin_2), U6.24 (REFCOM); no longer J5.1 (Pin_1), J6.1 (Pin_1), J7.1 (Pin_1), J8.1 (Pin_1), U6.15 (IOVDD)
- net at C33.2, C34.1, R4.1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: now also D2.1 (K); no longer L1.2, U3.1 (SW)
- new net: D2.2 (A), L1.2, U3.1 (SW)
Other:
- moved on the sheet: C38, L1, U3

Commit message: WIP
Parts:
- removed C45: 100 nF, >10V, X6S, Capacitor_SMD:C_0402_1005Metric, symbol Device:C_Small
- removed C46: 330 nF, Capacitor_SMD:C_0603_1608Metric, symbol Device:C_Small
- removed C47: 1 uF, >10V, X5R, Capacitor_SMD:C_0402_1005Metric, symbol Device:C_Small
- removed U2: 74HCT4066PW, Package_SO:SO-14_3.9x8.65mm_P1.27mm, symbol Analog_Switch:CD4066BM
- removed unit 2 of U2
- removed unit 3 of U2
- removed unit 4 of U2
- removed unit 5 of U2
- removed U6: ADS124S08IPBSR, Package_QFP:LQFP-32_5x5mm_P0.5mm, symbol ADS124S08IRHBR:ADS124S08IRHBR
- added C16, C37, C41, C43: 10 µF, Capacitor_SMD:C_0805_2012Metric, symbol Device:C_Small
- added C17, C18, C40, C42, C44: 100 nF, >10V, X6S, Capacitor_SMD:C_0402_1005Metric, symbol Device:C_Small
- added J11, J12: Conn_01x02, Connector_PinHeader_2.54mm:PinHeader_1x02_P2.54mm_Vertical, symbol Connector_Generic:Conn_01x02
- added Q7, Q8, Q9: DMN63D8LDW, PCM_Package_TO_SOT_SMD_AKL:SOT-363_SC-70-6, symbol PCM_Transistor_MOSFET_AKL:DMN63D8LDW
- added R29, R30, R31: 10K, Resistor_SMD:R_0402_1005Metric, symbol Device:R_Small
- added U2, U5: NAU7802SGI, PCM_Package_SO_AKL:SOP-16_4.4x10.4mm_P1.27mm, symbol NAU7802:NAU7802SGI
- C13: LCSC C711044 -> (none)
- C19: value 10nF -> 100 nF, >10V, X6S; LCSC C15195 -> C1525
- C20, C34, C36, C39: value 10µF -> 10 µF
- R20, R21, R22, R23, R24, R25, R26: value 47R -> 10K; LCSC C25118 -> C25744
- R27, R28: value 100R -> 10K; LCSC C25076 -> C25744
Connections:
- net EXCITATION2 is gone; now on net NAU7802_1_AVDD: J6.1 (Pin_1)
- net EXCITATION4 is gone; now on net NAU7802_2_AVDD: J8.1 (Pin_1)
- net +3V3: now also R20.1, R22.1, R24.1, R26.1, R28.1, Q7.2 (G1), Q7.5 (G2), Q8.2 (G1), Q8.5 (G2), Q9.2 (G1), Q9.5 (G2), R30.1
- net AVCC: now also R21.1, R23.1, R25.1, C16.2, C17.2, C42.2, C43.2, R29.1, R31.1, U2.15 (DVDD), U5.15 (DVDD)
- net GND: now also C19.2, C16.1, C17.1, C18.1, C37.1, C40.1, C41.1, C42.1, C43.1, C44.2, J11.2 (Pin_2), J12.2 (Pin_2), U2.7 (REFN), U2.8 (AVSS), U2.9 (DVSS), U5.7 (REFN), U5.8 (AVSS), U5.9 (DVSS); no longer R28.1
- net LOAD_CELL_1_N: now also U2.4 (VIN2N)
- net LOAD_CELL_1_P: now also U2.5 (VIN2P)
- net LOAD_CELL_2_N: now also U2.2 (VIN1N)
- net LOAD_CELL_2_P: now also U2.3 (VIN1P)
- net LOAD_CELL_3_N: now also U5.4 (VIN2N)
- net LOAD_CELL_3_P: now also U5.5 (VIN2P)
- net LOAD_CELL_4_N: now also U5.2 (VIN1N)
- net LOAD_CELL_4_P: now also U5.3 (VIN1P)
- net NAU7802_1_SDIO_3V3: now reaches U2.13 (GPIO10)
- net NAU7802_1_SDIO_3V3: now also R20.2, Q7.1 (S1)
- net NAU7802_1_SCLK_3V3: now reaches U2.14 (GPIO11)
- net NAU7802_1_SCLK_3V3: now also R22.2, Q7.4 (S2)
- net USER_BUTTON_1: now reaches U2.37 (GPIO25)
- net USER_BUTTON_1: now also J11.1 (Pin_1)
- net ADS124S08_CS: no longer names the net of U2.11 (GPIO8)
- net ADS124S08_CS: no longer R25.2
- net ADS124S08_DRDY renamed NAU7802_1_SDIO_5V
- net NAU7802_1_SDIO_5V: now also Q7.6 (D1), U2.14 (SDIO); no longer U2.5 (GPIO3)
- net ADS124S08_MISO: no longer names the net of U2.6 (GPIO4)
- net ADS124S08_MISO: no longer R22.2
- net ADS124S08_MOSI renamed NAU7802_1_DRDY_3V3
- net NAU7802_1_DRDY_3V3: now also Q8.1 (S1)
- net ADS124S08_RESETn renamed NAU7802_2_SDIO_3V3
- net NAU7802_2_SDIO_3V3: now also R26.2, Q9.1 (S1); no longer R20.2
- net ADS124S08_SCLK renamed NAU7802_1_SCLK_5V
- net NAU7802_1_SCLK_5V: now also Q7.3 (D2), U2.13 (SCLK); no longer U2.8 (GPIO6)
- net ADS124S08_START_SYNC: no longer names the net of U2.12 (GPIO9)
- net ADS124S08_START_SYNC: no longer R26.2
- net EXCITATION1 renamed NAU7802_1_AVDD
- net NAU7802_1_AVDD: now also C18.2, C37.2, U2.1 (REFP), U2.16 (AVDD/LDO)
- net EXCITATION1_EN: no longer names the net of U2.18 (GPIO15)
- net EXCITATION2_EN: no longer names the net of U2.17 (GPIO14)
- net EXCITATION3 renamed NAU7802_2_AVDD
- net NAU7802_2_AVDD: now also C40.2, C41.2, U5.1 (REFP), U5.16 (AVDD/LDO)
- net EXCITATION3_EN: no longer names the net of U2.16 (GPIO13)
- net EXCITATION4_EN renamed USER_BUTTON_2
- net USER_BUTTON_2: now also J12.1 (Pin_1)
- net REFN0 renamed NAU7802_2_SCLK_3V3
- net NAU7802_2_SCLK_3V3: now also U2.5 (GPIO3), Q9.4 (S2); no longer C19.2
- net REFP0: no longer names the net of C19.1
- net REFP0: now also U5.6 (VBG); no longer R27.2
- new net: C44.1, U2.6 (VBG)
- new net NAU7802_1_DRDY_5V: Q8.6 (D1), R25.2, U2.12 (DRDY)
- new net NAU7802_2_DRDY_3V3: Q8.4 (S2), R30.2, U2.8 (GPIO6)
- new net NAU7802_2_DRDY_5V: Q8.3 (D2), R31.2, U5.12 (DRDY)
- new net NAU7802_2_SCLK_5V: Q9.3 (D2), R29.2, U5.13 (SCLK)
- new net NAU7802_2_SDIO_5V: Q9.6 (D1), R27.2, U5.14 (SDIO)
Other:
- note added: "I2C0"

Commit message: WIP
Parts:
- removed U6: ADP7118, Package_TO_SOT_SMD:TSOT-23-5, symbol Regulator_Linear:ADP7118ACPZN
- added C45: 1 nF, Capacitor_SMD:C_0402_1005Metric, symbol Device:C_Small
- added U7: ADM7170ACPZ-1.8-R7, ADM7170ACPZ-1:SON50P300X300X80-9N, symbol ADM7170ACPZ-1.8-R7:ADM7170ACPZ-1.8-R7
- C10, C11: value 5.1 nF -> X nF
- C13: value 51 nF -> 10X nF
- C16, C20, C34, C36, C37, C39, C41, C43: value 10 µF -> 10 µF, >10V, X5R
- R15, R16: value 6K04 1% -> Y R
- R19: value 10K -> 6K8; footprint Resistor_SMD:R_0402_1005Metric -> Resistor_SMD:R_0603_1608Metric; LCSC C25744 -> C23212
- R4: value 47K -> 27K; footprint Resistor_SMD:R_0402_1005Metric -> Resistor_SMD:R_0603_1608Metric; LCSC C25792 -> C22967
Connections:
- net AVCC: now also U7.1 (VOUT), U7.2 (VOUT), U7.3 (SENSE)
- net GND: now also C45.2, U7.6 (GND), U7.9 (EXP)
- net at C33.2, C34.1, D2.1 (K)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: now also U7.5 (EN), U7.7 (VIN), U7.8 (VIN)
- new net: C45.1, U7.4 (SS)
Other:
- moved on the sheet: C20, C35

Commit message: Final version sent to manufacturing
Parts:
- removed D4: KT-0603W, LED_SMD:LED_0603_1608Metric, symbol Device:LED
- removed R12: 120R, Resistor_SMD:R_0402_1005Metric, symbol Device:R_Small
- added D4 (x2): KT-0603W, LED_SMD:LED_0603_1608Metric, symbol Device:LED
- added JP1: SolderJumper_3_Bridged12, Jumper:SolderJumper-3_P1.3mm_Bridged12_RoundedPad1.0x1.5mm, symbol Jumper:SolderJumper_3_Bridged12
- added R12 (x2): 120R, Resistor_SMD:R_0402_1005Metric, symbol Device:R_Small
- added TP1, TP2: TestPoint, TestPoint:TestPoint_Pad_D2.0mm, symbol Connector:TestPoint
- added TP3, TP4, TP5, TP6: TestPoint, TestPoint:TestPoint_Pad_D1.0mm, symbol Connector:TestPoint
- C10, C11: value X nF -> DNF; Comment (none) -> Hand solder; now not fitted
- C10, C11: value X nF -> 680 pF, C0G; LCSC (none) -> C326939
- C13: value 10X nF -> 100 nF, C0G; Comment (none) -> Hand solder; LCSC (none) -> C97946
- C13: value 10X nF -> 680 pF, C0G; LCSC (none) -> C326939
- C37, C41: value 10 µF, >10V, X5R -> 1 uF, >10V, X5R; footprint Capacitor_SMD:C_0805_2012Metric -> Capacitor_SMD:C_0402_1005Metric; LCSC C440198 -> C52923
- Q7, Q8, Q9: Comment (none) -> Extended
- R15, R16: value Y R -> DNF; now not fitted
- R15, R16: value Y R -> 51R, Precision; Comment (none) -> Hand solder; LCSC (none) -> C2828901
- SW1, SW2: LCSC (none) -> C271750
Connections:
- net +3V3: now also JP1.3 (B)
- net AVCC: now also JP1.2 (C); no longer C20.1, C35.2, U7.1 (VOUT), U7.2 (VOUT), U7.3 (SENSE)
- net GND: now also D4.1 (K), D4.1 (K)
- net at C33.2, C34.1, D2.1 (K)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: now also TP1.1
- net at U2.17 (GPIO14): now also R12.1
- net at U2.18 (GPIO15): now also R12.1
- net at U2.27 (GPIO16): now also TP3.1
- net at U2.28 (GPIO17): now also TP4.1
- net at U2.29 (GPIO18): now also TP5.1
- net at U2.30 (GPIO19): now also TP6.1
- net LOAD_CELL_1_N renamed LOAD_CELL_ADC1_2_N
- net LOAD_CELL_1_P renamed LOAD_CELL_ADC1_2_P
- net LOAD_CELL_2_N renamed LOAD_CELL_ADC1_1_N
- net LOAD_CELL_2_P renamed LOAD_CELL_ADC1_1_P
- net LOAD_CELL_3_N renamed LOAD_CELL_ADC2_2_N
- net LOAD_CELL_3_P renamed LOAD_CELL_ADC2_2_P
- net LOAD_CELL_4_N renamed LOAD_CELL_ADC2_1_N
- net LOAD_CELL_4_P renamed LOAD_CELL_ADC2_1_P
- new net: D4.2 (A), R12.2 (x2)
- new net +5VA: C20.1, C35.2, JP1.1 (A), TP2.1, U7.1 (VOUT), U7.2 (VOUT), U7.3 (SENSE)
- no-connect marks 25 -> 20

Commit message: WIP
Parts:
- added J13: BM03B-SRSS-TBLFSN, CONN_BM03B-SRSS-TBLFSN_JST, symbol BM03B-SRSS-TB_LF__SN_:BM03B-SRSS-TBLFSN
- added JP2, JP3: SolderJumper_3_Bridged12, Jumper:SolderJumper-3_P1.3mm_Bridged12_RoundedPad1.0x1.5mm, symbol Jumper:SolderJumper_3_Bridged12
- added R33, R34: 100R, Resistor_SMD:R_0402_1005Metric, symbol Device:R_Small
- added TP10, TP11, TP12, TP7, TP8, TP9: TestPoint_Small, TestPoint:TestPoint_Pad_D1.0mm, symbol Connector:TestPoint_Small
Connections:
- net GND: now also J13.2
- net NAU7802_1_DRDY_5V: now also TP12.1
- net NAU7802_1_SCLK_3V3: now also JP3.2 (C); no longer U2.14 (GPIO11)
- net NAU7802_1_SCLK_5V: now also TP11.1
- net NAU7802_1_SDIO_3V3: now also JP2.2 (C); no longer U2.13 (GPIO10)
- net NAU7802_1_SDIO_5V: now also TP10.1
- net NAU7802_2_DRDY_5V: now also TP9.1
- net NAU7802_2_SCLK_5V: now also TP8.1
- net NAU7802_2_SDIO_5V: now also TP7.1
- net RP2040_SWCLK: now also R33.1
- net RP2040_SWD: now also R34.2
- net NAU7802_1_SDIO_3V3_ALT_B: now reaches U2.11 (GPIO8)
- net NAU7802_1_SDIO_3V3_ALT_B: now also JP2.3 (B)
- net NAU7802_1_SCLK_3V3_ALT_B: now reaches U2.12 (GPIO9)
- net NAU7802_1_SCLK_3V3_ALT_B: now also JP3.3 (B)
- new net: J13.1, R33.2
- new net: J13.3, R34.1
- new net NAU7802_1_SCLK_3V3_ALT_A: JP3.1 (A), U2.14 (GPIO11)
- new net NAU7802_1_SDIO_3V3_ALT_A: JP2.1 (A), U2.13 (GPIO10)
- no-connect marks 20 -> 18

Commit message: WIP
Parts:
- removed D4 (x2): KT-0603W, LED_SMD:LED_0603_1608Metric, symbol Device:LED
- removed J1: USB_B_Micro, Connector_USB:USB_Micro-B_Molex-105133-0001, symbol Connector:USB_B_Micro
- removed J11, J12: Conn_01x02, Connector_PinHeader_2.54mm:PinHeader_1x02_P2.54mm_Vertical, symbol Connector_Generic:Conn_01x02
- removed JP2, JP3: SolderJumper_3_Bridged12, Jumper:SolderJumper-3_P1.3mm_Bridged12_RoundedPad1.0x1.5mm, symbol Jumper:SolderJumper_3_Bridged12
- removed Q9: DMN63D8LDW, PCM_Package_TO_SOT_SMD_AKL:SOT-363_SC-70-6, symbol PCM_Transistor_MOSFET_AKL:DMN63D8LDW
- removed R12 (x2): 120R, Resistor_SMD:R_0402_1005Metric, symbol Device:R_Small
- removed TP1, TP2: TestPoint, TestPoint:TestPoint_Pad_D2.0mm, symbol Connector:TestPoint
- removed TP10, TP11, TP12, TP7, TP8, TP9: TestPoint_Small, TestPoint:TestPoint_Pad_D1.0mm, symbol Connector:TestPoint_Small
- removed TP3, TP4, TP5, TP6: TestPoint, TestPoint:TestPoint_Pad_D1.0mm, symbol Connector:TestPoint
- removed U4: AMS1117-3.3, Package_TO_SOT_SMD:SOT-223-3_TabPin2, symbol Regulator_Linear:AMS1117-3.3
- added C12: 1 uF, >6.3V, X5R, Capacitor_SMD:C_0402_1005Metric, symbol Device:C
- added C24: 100 nF, >10V, X6S, Capacitor_SMD:C_0402_1005Metric, symbol Device:C_Small
- added C28: 22 uF, 6.3V, X5R, Capacitor_SMD:C_0603_1608Metric, symbol Device:C_Small
- added D4 (x2): KT-0603W, LED_SMD:LED_0603_1608Metric, symbol Device:LED
- added J1: Molex_527461871, CON_527461871_MOL:CON_527461871_MOL, symbol ADS1119:EyeSPI
- added J13: Conn_02x05_Odd_Even, Connector_PinHeader_1.27mm:PinHeader_2x05_P1.27mm_Vertical_SMD, symbol Connector_Generic:Conn_02x05_Odd_Even
- added J14: USB_C_Receptacle_USB2.0, Connector_USB:USB_C_Receptacle_G-Switch_GT-USB-7010ASV, symbol Connector:USB_C_Receptacle_USB2.0
- added J15: Conn_01x03, Connector_PinHeader_2.54mm:PinHeader_1x03_P2.54mm_Vertical_SMD_Pin1Left, symbol Connector_Generic:Conn_01x03
- added J3: Conn_02x03_Odd_Even, Connector_PinHeader_1.27mm:PinHeader_2x03_P1.27mm_Vertical_SMD, symbol Connector_Generic:Conn_02x03_Odd_Even
- added NT1, NT2: NetTie_2, NetTie:NetTie-2_SMD_Pad0.5mm, symbol Device:NetTie_2
- added Q7: DMN63D8LDW, PCM_Package_TO_SOT_SMD_AKL:SOT-363_SC-70-6, symbol PCM_Transistor_MOSFET_AKL:DMN63D8LDW
- added R12 (x2): 120R, Resistor_SMD:R_0402_1005Metric, symbol Device:R_Small
- added R35: 2K7 1%, Resistor_SMD:R_0402_1005Metric, symbol Device:R_Small
- added R36: 10K, Resistor_SMD:R_0402_1005Metric, symbol Device:R_Small
- added R38, R39: 5K1, Resistor_SMD:R_0402_1005Metric, symbol Device:R_Small
- added R9: 10K, Resistor_SMD:R_0402_1005Metric, symbol Device:R
- added SW1, SW2: SW_Push, ul_PTS815-SJM-250-SMTR-LFS:SW4_PTS815 SJM 250 SMTR LFS_CNK, symbol Switch:SW_Push
- added U4: LTC4316CMS_PBF, Package_SO:MSOP-10_3x3mm_P0.5mm, symbol LTC4316CMS_PBF:LTC4316CMS_PBF
- added U6: ESP32-C6-MINI-1/U, PCM_Espressif:ESP32-C6-MINI-1, symbol PCM_Espressif:ESP32-C6-MINI-1/U
- added U8: FE1.1s (Rev B), Package_SO:SSOP-28_3.9x9.9mm_P0.635mm, symbol Interface_USB:FE1.1s
- added Y3: 12MHz, Crystal:Crystal_SMD_3225-4Pin_3.2x2.5mm, symbol Device:Crystal_GND24_Small
- J13: LCSC (none) -> C160389
- JP1: footprint Jumper:SolderJumper-3_P1.3mm_Bridged12_RoundedPad1.0x1.5mm -> Jumper:SolderJumper-3_P1.3mm_Bridged2Bar12_RoundedPad1.0x1.5mm_NumberLabels; Comment (none) -> No solder; now left out of the parts list
- R26: value 10K -> 976K; LCSC C25744 -> C227280
- R28: value 10K -> 182K; LCSC C25744 -> C327365
- R33, R34: LCSC (none) -> C25076
- R5, R6: footprint Resistor_SMD:R_0603_1608Metric -> Resistor_SMD:R_0402_1005Metric
- SW1, SW2: footprint Button_Switch_SMD:SW_SPST_Omron_B3FS-100xP -> ul_PTS815-SJM-250-SMTR-LFS:SW4_PTS815 SJM 250 SMTR LFS_CNK
Connections:
- net NAU7802_1_SCLK_3V3_ALT_A is gone; now on net NAU7802_1_SCLK_3V3: U2.14 (GPIO11)
- net NAU7802_1_SDIO_3V3_ALT_A is gone; now on net NAU7802_1_SDIO_3V3: U2.13 (GPIO10)
- net +3V3: now also C24.2, C28.2, J1.1 (Vcc), J13.1 (Pin_1), J3.2 (Pin_2), NT1.2, NT2.2, R36.2, R9.1, U4.4 (VCC), U4.5 (ENABLE), U6.22 (GPIO8), U6.3 (3V3), U8.21 (VD33_O), U8.26 (OVCJ); no longer J5.2, J5.2, R28.1
- net +5VA: now also C16.2, C17.2, C42.2, C43.2, R21.1, R23.1, R25.1, R27.1, R29.1, R31.1, U2.15 (DVDD), U5.15 (DVDD); no longer JP1.1 (A)
- net GND: now also JP1.1 (A), R28.2, C12.1, C24.1, C28.1, D4.1 (K), D4.1 (K), J1.3 (GND), J13.3 (Pin_3), J13.5 (Pin_5), J13.9 (Pin_9), J14.A1 (GND), J14.A12 (GND), J14.B1 (GND), J14.B12 (GND), J14.S1 (SHIELD), J15.3 (Pin_3), J3.4 (Pin_4), Q7.1 (S1), Q7.4 (S2), R35.1, R38.2, R39.2, SW1.2, SW2.2, U4.1 (GND), U4.2 (XORH), U6.1 (GND), U6.11 (GND), U6.14 (GND), U6.2 (GND), U6.36 (GND), U6.37 (GND), U6.38 (GND), U6.39 (GND), U6.40 (GND), U6.41 (GND), U6.42 (GND), U6.43 (GND), U6.44 (GND), U6.45 (GND), U6.46 (GND), U6.47 (GND), U6.48 (GND), U6.49 (GND), U6.50 (GND), U6.51 (GND), U6.52 (GND), U6.53 (GND), U8.1 (VSS), U8.19 (BUSJ), Y3.2, Y3.4
- net NAU7802_1_DRDY_3V3: now also U2.7 (GPIO5); no longer U2.9 (GPIO7)
- net NAU7802_1_SCLK_3V3: now also U4.10 (SCLIN)
- net NAU7802_1_SDIO_3V3: now also U4.7 (SDAIN)
- net NAU7802_2_DRDY_3V3: now also U2.6 (GPIO4); no longer U2.8 (GPIO6)
- net NAU7802_2_SCLK_5V: now also U4.9 (SCLOUT)
- net NAU7802_2_SDIO_5V: now also U4.8 (SDAOUT)
- net QWIIC_SCL: now also J1.13 (SCL)
- net QWIIC_SDA: now also J1.14 (SDA)
- net RP2040_BOOTSEL: now also Q7.6 (D1)
- net RP2040_RESETn: now also Q7.3 (D2)
- net RP2040_USB_POST_R_DN: now also U8.10 (DM1)
- net RP2040_USB_POST_R_DP: now also U8.11 (DP1)
- net RP2040_ESP32_GP2: now reaches U2.18 (GPIO15)
- net RP2040_ESP32_GP2: now also U6.29 (GPIO23)
- net EYESPI_MOSI: now reaches U2.30 (GPIO19)
- net EYESPI_MOSI: now also J1.5 (MOSI)
- net EYESPI_DISP_CS: now reaches U2.28 (GPIO17)
- net EYESPI_DISP_CS: now also J1.9 (DISP_CS)
- net USER_1: now reaches U2.16 (GPIO13)
- net USER_1: now also J15.1 (Pin_1)
- net RP2040_ESP32_GP1: now reaches U2.17 (GPIO14)
- net RP2040_ESP32_GP1: now also U6.28 (GPIO22)
- net EYESPI_MISO: now reaches U2.27 (GPIO16)
- net EYESPI_MISO: now also J1.6 (MISO)
- net EYESPI_SCK: now reaches U2.29 (GPIO18)
- net EYESPI_SCK: now also J1.4 (SCK)
- net EYESPI_RES: now reaches U2.34 (GPIO22)
- net EYESPI_RES: now also J1.8 (RESET)
- net EYESPI_DC: now reaches U2.35 (GPIO23)
- net EYESPI_DC: now also J1.7 (DC)
- net EYESPI_BUSY_TE: now reaches U2.36 (GPIO24)
- net EYESPI_BUSY_TE: now also J1.16 (BUSY/TE)
- net EYESPI_BL: now reaches U2.38 (GPIO26_ADC0)
- net EYESPI_BL: now also J1.2 (BACKLIGHT)
- net EYESPI_TS_CS: now reaches U2.39 (GPIO27_ADC1)
- net EYESPI_TS_CS: now also J1.12 (TS_CS)
- net EYESPI_MEM_CS: now reaches U2.40 (GPIO28_ADC2)
- net EYESPI_MEM_CS: now also J1.11 (MEM_CS)
- net EYESPI_SD_CS: now reaches U2.41 (GPIO29_ADC3)
- net EYESPI_SD_CS: now also J1.10 (SD_CS)
- removed net AVCC: C16.2, C17.2, C42.2, C43.2, JP1.2 (C), R21.1, R23.1, R25.1, R27.1, R29.1, R31.1, U2.15 (DVDD), U5.15 (DVDD)
- net NAU7802_1_SCLK_3V3_ALT_B renamed RP2040_ESP32_RX
- net RP2040_ESP32_RX: now also U6.12 (GPIO0/ADC1_CH0/XTAL_32K_P)
- net NAU7802_1_SDIO_3V3_ALT_B renamed RP2040_ESP32_TX
- net RP2040_ESP32_TX: now also U6.13 (GPIO1/ADC1_CH1/XTAL_32K_N)
- net NAU7802_2_SCLK_3V3 renamed EYESPI_GP2
- net EYESPI_GP2: now also J1.18 (GPIO2); no longer R28.2
- net NAU7802_2_SDIO_3V3: no longer names the net of R26.2
- net NAU7802_2_SDIO_3V3: now also R28.1, U4.3 (XORL); no longer U2.4 (GPIO2)
- net RP2040_USB_VBUS renamed USB_VBUS
- net USB_VBUS: now also J14.A4 (VBUS), J14.A9 (VBUS), J14.B4 (VBUS), J14.B9 (VBUS), U8.18 (VBUSM), U8.20 (VDD5)
- net USER_BUTTON_1 renamed EYESPI_INT
- net EYESPI_INT: now also J1.15 (INT)
- net USER_BUTTON_2 renamed USER_2
- net USER_2: now also J15.2 (Pin_2)
- new net: U8.3 (XIN), Y3.1
- new net: U8.2 (XOUT), Y3.3
- new net: J14.A5 (CC1), R39.1
- new net: R12.1, U2.8 (GPIO6)
- new net: D4.2 (A), R12.2 (x2)
- new net: J14.B5 (CC2), R38.1
- new net: R35.2, U8.14 (REXT)
- new net: R36.1, U8.17 (~{XRSTJ})
- new net ESP32_BOOTSEL_RP2040: Q7.2 (G1), U6.5 (GPIO2/ADC1_CH2)
- new net ESP32_DISABLE_RP2040: Q7.5 (G2), U6.6 (GPIO3/ADC1_CH3)
- new net ESP32_EN: C12.2, J13.10 (Pin_10), J3.1 (Pin_1), R9.2, SW2.1, U6.8 (EN/CHIP_PU)
- new net ESP32_GPIO0: J3.6 (Pin_6), R12.1, SW1.1, U6.23 (GPIO9)
- new net ESP32_JTAG_SELECT: JP1.2 (C), U6.20 (GPIO15)
- new net ESP32_TCK: J13.4 (Pin_4), U6.15 (MTCK/GPIO6/ADC1_CH6)
- new net ESP32_TDI: J13.8 (Pin_8), U6.10 (MTDI/GPIO5/ADC1_CH5)
- new net ESP32_TDO: J13.6 (Pin_6), U6.16 (MTDO/GPIO7)
- new net ESP32_TMS: J13.2 (Pin_2), U6.9 (MTMS/GPIO4/ADC1_CH4)
- new net ESP32_U0RXD: J3.5 (Pin_5), U6.30 (U0RXD/GPIO17)
- new net ESP32_U0TXD: J3.3 (Pin_3), U6.31 (U0TXD/GPIO16)
- new net ESP32_USB_DN: U6.17 (GPIO12/USB_D-), U8.8 (DM2)
- new net ESP32_USB_DP: U6.18 (GPIO13/USB_D+), U8.9 (DP2)
- new net EYESPI_GP1: J1.17 (GPIO1), U2.4 (GPIO2)
- new net QWIIC_VIN1: J5.2, NT1.1
- new net QWIIC_VIN2: J5.2, NT2.1
- new net RP2040_SERIAL_BOOT: U2.9 (GPIO7), U6.19 (GPIO14)
- new net USB_UPSTREAM_DN: J14.A7 (D-), J14.B7 (D-), U8.15 (DMU)
- new net USB_UPSTREAM_DP: J14.A6 (D+), J14.B6 (D+), U8.16 (DPU)
- no-connect marks 18 -> 27
Other:
- note added: "EyeSPI Connector"
- moved on the sheet: Q8B, R27, R29, R30, R31, SW1, SW2

Commit message: R3B
Parts:
- removed Q7: DMN63D8LDW, PCM_Package_TO_SOT_SMD_AKL:SOT-363_SC-70-6, symbol PCM_Transistor_MOSFET_AKL:DMN63D8LDW
- removed R22, R23: 10K, Resistor_SMD:R_0402_1005Metric, symbol Device:R_Small
- removed U6: ESP32-C6-MINI-1/U, PCM_Espressif:ESP32-C6-MINI-1, symbol PCM_Espressif:ESP32-C6-MINI-1/U
- added C49, C50: 1 uF, >10V, X5R, Capacitor_SMD:C_0402_1005Metric, symbol Device:C_Small
- added JP2, JP3, JP4: SolderJumper_3_Bridged12, Jumper:SolderJumper-3_P1.3mm_Bridged2Bar12_RoundedPad1.0x1.5mm_NumberLabels, symbol Jumper:SolderJumper_3_Bridged12
- added Q2, Q3: 2N7002, Package_TO_SOT_SMD:SOT-23-3, symbol PCM_Transistor_MOSFET_AKL:2N7002
- added R10, R9: 10K, Resistor_SMD:R_1206_3216Metric, symbol Device:R_Small
- added U6: TLV75733PDBVR, Package_TO_SOT_SMD:SOT-23-5, symbol TLV75733PDBVR:TLV75733PDBVR
- added U9: ESP32-C6-WROOM-1, PCM_Espressif:ESP32-C6-WROOM-1, symbol PCM_Espressif:ESP32-C6-WROOM-1
- C12: footprint Capacitor_SMD:C_0402_1005Metric -> Capacitor_SMD:C_1206_3216Metric; LCSC C426073 -> C1848
- C24: footprint Capacitor_SMD:C_0402_1005Metric -> Capacitor_SMD:C_1206_3216Metric; LCSC C1525 -> C24497
- C28: footprint Capacitor_SMD:C_0603_1608Metric -> Capacitor_SMD:C_1206_3216Metric; LCSC C59461 -> C12891
- C39: value 10 µF, >10V, X5R -> 1 uF, >10V, X5R; footprint Capacitor_SMD:C_0805_2012Metric -> Capacitor_SMD:C_0402_1005Metric; LCSC C440198 -> C52923
- D4: value KT-0603W -> KT-1206R; footprint LED_SMD:LED_0603_1608Metric -> LED_SMD:LED_1206_3216Metric; LCSC C2290 -> C49018
- J1: value Molex_527461871 -> Molex 0527451897; LCSC C3169221 -> C7153842
- R12: footprint Resistor_SMD:R_0402_1005Metric -> Resistor_SMD:R_1206_3216Metric; LCSC C25079 -> C17909
- R19: footprint Resistor_SMD:R_0603_1608Metric -> Resistor_SMD:R_0402_1005Metric; LCSC C23212 -> C25917
- R26: value 976K -> 10K; LCSC C227280 -> C25744
- R28: value 182K -> 4K7; LCSC C327365 -> C25900
- R4: footprint Resistor_SMD:R_0603_1608Metric -> Resistor_SMD:R_0402_1005Metric; LCSC C22967 -> C25771
- R5, R6: footprint Resistor_SMD:R_0402_1005Metric -> Resistor_SMD:R_0603_1608Metric
- R9: footprint Resistor_SMD:R_0402_1005Metric -> Resistor_SMD:R_1206_3216Metric; LCSC C25744 -> C17902
- SW1, SW2: LCSC C271750 -> C918859
Connections:
- net +3V3: now also C49.1, JP4.3 (B), U6.5 (OUT), U9.10 (GPIO8), U9.2 (3V3)
- net ESP32_BOOTSEL_RP2040: now also Q2.1 (G), R9.2, U9.27 (GPIO2/ADC1_CH2)
- net ESP32_DISABLE_RP2040: now also Q3.1 (G), R10.2, U9.26 (GPIO3/ADC1_CH3)
- net ESP32_EN: now also U9.3 (EN/CHIP_PU)
- net ESP32_JTAG_SELECT: now also U9.23 (GPIO15)
- net ESP32_TCK: now also U9.6 (MTCK/GPIO6/ADC1_CH6)
- net ESP32_TDI: now also U9.5 (MTDI/GPIO5/ADC1_CH5)
- net ESP32_TDO: now also U9.7 (MTDO/GPIO7)
- net ESP32_TMS: now also U9.4 (MTMS/GPIO4/ADC1_CH4)
- net ESP32_U0RXD: now also U9.24 (U0RXD/GPIO17)
- net ESP32_U0TXD: now also U9.25 (U0TXD/GPIO16)
- net ESP32_USB_DN: now also U9.13 (GPIO12/USB_D-)
- net ESP32_USB_DP: now also U9.14 (GPIO13/USB_D+)
- net EYESPI_BL: now also U2.41 (GPIO29_ADC3); no longer U2.38 (GPIO26_ADC0)
- net EYESPI_BUSY_TE: now also U2.27 (GPIO16); no longer U2.36 (GPIO24)
- net EYESPI_DC: now also U2.37 (GPIO25); no longer U2.35 (GPIO23)
- net EYESPI_DISP_CS: now also U2.35 (GPIO23); no longer U2.28 (GPIO17)
- net EYESPI_GP1: now also U2.17 (GPIO14); no longer U2.4 (GPIO2)
- net EYESPI_GP2: now also U2.18 (GPIO15); no longer U2.5 (GPIO3)
- net EYESPI_INT: now also U2.28 (GPIO17); no longer U2.37 (GPIO25)
- net EYESPI_MEM_CS: now also U2.32 (GPIO21); no longer U2.40 (GPIO28_ADC2)
- net EYESPI_MISO: now also U2.40 (GPIO28_ADC2); no longer U2.27 (GPIO16)
- net EYESPI_MOSI: now also U2.39 (GPIO27_ADC1); no longer U2.30 (GPIO19)
- net EYESPI_RES: now also U2.36 (GPIO24); no longer U2.34 (GPIO22)
- net EYESPI_SCK: now also U2.38 (GPIO26_ADC0); no longer U2.29 (GPIO18)
- net EYESPI_SD_CS: now also U2.34 (GPIO22); no longer U2.41 (GPIO29_ADC3)
- net EYESPI_TS_CS: now also U2.31 (GPIO20); no longer U2.39 (GPIO27_ADC1)
- net GND: now also C49.2, C50.2, JP4.1 (A), Q2.2 (S), Q3.2 (S), R10.1, R9.1, U6.2 (GND), U9.1 (GND), U9.12 (GPIO11), U9.28 (GND), U9.29 (GND); no longer U8.19 (BUSJ)
- net NAU7802_1_DRDY_3V3: now also U2.14 (GPIO11); no longer U2.7 (GPIO5)
- net NAU7802_1_SCLK_3V3: now also U2.12 (GPIO9), JP3.3 (B); no longer U2.14 (GPIO11)
- net NAU7802_1_SDIO_3V3: now also U2.11 (GPIO8), JP2.3 (B); no longer U2.13 (GPIO10)
- net NAU7802_2_DRDY_3V3: now also U2.13 (GPIO10); no longer U2.6 (GPIO4)
- net QWIIC_SCL: now also U2.30 (GPIO19), JP3.1 (A); no longer J5.4, U2.32 (GPIO21)
- net QWIIC_SDA: now also U2.29 (GPIO18), JP2.1 (A); no longer J5.3, U2.31 (GPIO20)
- net RP2040_BOOTSEL: now also Q2.3 (D)
- net RP2040_ESP32_GP1: now also U2.4 (GPIO2), U9.20 (GPIO22); no longer U2.17 (GPIO14)
- net RP2040_ESP32_GP2: now also U2.5 (GPIO3), U9.21 (GPIO23); no longer U2.18 (GPIO15)
- net RP2040_ESP32_RX: now also U2.7 (GPIO5), U9.9 (GPIO1/ADC1_CH1/XTAL_32K_N); no longer U2.12 (GPIO9)
- net RP2040_ESP32_TX: now also U2.6 (GPIO4), U9.8 (GPIO0/ADC1_CH0/XTAL_32K_P); no longer U2.11 (GPIO8)
- net RP2040_RESETn: now also Q3.3 (D)
- net RP2040_SERIAL_BOOT: now also U9.11 (GPIO10)
- net USB_VBUS: now also C50.1, U6.1 (IN), U6.3 (EN); no longer U8.20 (VDD5)
- net RP2040_LED: now reaches R12.1, U2.8 (GPIO6)
- net ESP32_GPIO0 renamed ESP32_GPIO9
- net ESP32_GPIO9: now also U9.15 (GPIO9); no longer R12.1
- new net: JP4.2 (C), U8.19 (BUSJ)
- new net: R12.1, U9.16 (GPIO18)
- new net: J5.3, JP2.2 (C)
- new net: J5.4, JP3.2 (C)
Other:
- note added: "I2C1"
- note added: "SPI1"
- note added: "UART0"
- note added: "UART1"
- moved on the sheet: H1, H2, J5, R12
